File: Hardware/PCB_Atlas_Gauntlet/PCB_Atlas_Gauntlet.kicad_sch (KiCad schematic)
At the start: 40 parts, among them J1 Conn_01x02, J11 Conn_01x03, J13 Conn_01x03, J2 Conn_01x02, J3 Conn_01x03, J4 Conn_ST_STDC14, J5 Conn_01x03, J6 Conn_01x03, J7 Conn_01x03, J8 Conn_01x03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

Commit message: fix schematic
Parts:
- removed R22: 10k, Resistor_SMD:R_0402_1005Metric, symbol Device:R_Small
- removed SW6: SW_Push, Connector_JST:JST_XH_B2B-XH-AM_1x02_P2.50mm_Vertical, symbol Switch:SW_Push
- added C10, C11, C5, C6, C7, C8, C9: 10u, Capacitor_SMD:C_0603_1608Metric, symbol Device:C
- added C3: 47u, Capacitor_SMD:C_0805_2012Metric, symbol Device:C
- added C4: 220u, Capacitor_SMD:CP_Elec_8x10.5, symbol Device:C_Polarized_Small
- C1: footprint Capacitor_SMD:C_0402_1005Metric -> Capacitor_SMD:C_0603_1608Metric; MPN (none) -> 885 012 106 006
- J1: footprint Connector_AMASS:AMASS_XT30PW-M_1x02_P2.50mm_Horizontal -> Connector_AMASS:AMASS_XT30U-F_1x02_P5.0mm_Vertical
- SW1: footprint Connector_JST:JST_XH_B2B-XH-AM_1x02_P2.50mm_Vertical -> Button_Switch_SMD:SW_Push_1P1T_NO_CK_KSC7xxJ
Connections:
- net ADD_SEL_0 is gone; now on net LED_0: U3.14 (PB0)
- net BOOT_0 is gone; now on net GND: U3.31 (PH3)
- net RCC_CLK_IN is gone; now on net Servo_1: U3.6 (PA0)
- net +3.3V: now also C3.1
- net +5V: now also C10.1, C11.1, C5.1, C6.1, C7.1, C8.1, C9.1
- net Button_Mode: now also U3.3 (PC15); no longer U3.28 (PB5)
- net GND: now also C10.2, C11.2, C3.2, C4.2, C5.2, C6.2, C7.2, C8.2, C9.2
- net LED_0: no longer U3.2 (PC14)
- net LED_1: now also U3.15 (PB1); no longer U3.3 (PC15)
- net Servo_1: no longer U3.7 (PA1)
- net Servo_2: now also U3.7 (PA1); no longer U3.15 (PB1)
- net Servo_3: now also U3.8 (PA2); no longer U3.18 (PA8)
- net Servo_4: now also U3.9 (PA3); no longer U3.19 (PA9)
- net Servo_5: now also U3.12 (PA6); no longer U3.21 (PA11)
- net Switch_On_Off: now also U3.2 (PC14); no longer U3.27 (PB4)
- net VCC: now also C4.1
- net VCP_RX: now also U3.30 (PB7); no longer U3.9 (PA3)
- net VCP_TX: now also U3.29 (PB6); no longer U3.8 (PA2)
- net BTN_1: no longer names the net of U3.25 (PA15)
- net GPIO_LED_1 renamed NEOPIXEL_PWM_1
- net NEOPIXEL_PWM_1: now also U3.18 (PA8); no longer U3.29 (PB6)
- net GPIO_LED_2 renamed NEOPIXEL_PWM_2
- net NEOPIXEL_PWM_2: now also U3.19 (PA9); no longer U3.30 (PB7)
- no-connect marks 3 -> 12
Other:
- moved on the sheet: C15, C16, C17, C18, J1, J3, J5, J8

Commit message: MAJ_PCB
Connections:
- net VCC is gone; now on net +5V: C1.1, C4.1, J1.1 (Pin_1), U2.4, U2.5
Changed lines of the file:
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@@
 	(symbol
 		(lib_id "power:+5V")
+		(at 184.15 40.64 0)
+		(unit 1)
+		(exclude_from_sim no)
+		(in_bom yes)
+		(on_board yes)
+		(dnp no)
+		(fields_autoplaced yes)
+		(property "Reference" "#PWR03"
+			(at 184.15 44.45 0)
+			(effects
+				(font
+					(size 1.27 1.27)
+				)
+				(hide yes)
+			)
+		)
+		(property "Value" "+5V"
+			(at 184.15 35.56 0)
+			(effects
+				(font
+					(size 1.27 1.27)
+				)
+			)
+		)
+		(property "Footprint" ""
+			(at 184.15 40.64 0)
+			(effects
+				(font
+					(size 1.27 1.27)
+				)
+				(hide yes)
+			)
+		)
+		(property "Datasheet" ""
+			(at 184.15 40.64 0)
+			(effects
+				(font
+					(size 1.27 1.27)
+				)
+				(hide yes)
+			)
+		)
+		(property "Description" "Power symbol creates a global label with name \"+5V\""
+			(at 184.15 40.64 0)
+			(effects
+				(font
+					(size 1.27 1.27)
+				)
+				(hide yes)
+			)
+		)
+		(pin "1"
+		)
+		(instances
+			(project ""
+				(path "/61133cf5-41c1-41ca-a141-b2575d6d1c5c"
+					(reference "#PWR03")
+					(unit 1)
+				)
+			)
+		)
+	)
+	(symbol
+		(lib_id "power:+5V")
 		(at 34.29 173.99 270)
 		(unit 1)
@@
 	)
 	(symbol
+		(lib_id "power:+5V")
+		(at 208.28 22.86 0)
+		(unit 1)
+		(exclude_from_sim no)
+		(in_bom yes)
+		(on_board yes)
+		(dnp no)
+		(fields_autoplaced yes)
+		(property "Reference" "#PWR01"
+			(at 208.28 26.67 0)
+			(effects
+				(font
+					(size 1.27 1.27)
+				)
+				(hide yes)
+			)
+		)
+		(property "Value" "+5V"
+			(at 208.28 17.78 0)
+			(effects
+				(font
+					(size 1.27 1.27)
+				)
+			)
+		)
+		(property "Footprint" ""
+			(at 208.28 22.86 0)
+			(effects
+				(font
+					(size 1.27 1.27)
+				)
+				(hide yes)
+			)
+		)
+		(property "Datasheet" ""
+			(at 208.28 22.86 0)
+			(effects
+				(font
+					(size 1.27 1.27)
+				)
+				(hide yes)
+			)
+		)
+		(property "Description" "Power symbol creates a global label with name \"+5V\""
+			(at 208.28 22.86 0)
+			(effects
+				(font
+					(size 1.27 1.27)
+				)
+				(hide yes)
+			)
+		)
+		(pin "1"
+		)
+		(instances
+			(project ""
+				(path "/61133cf5-41c1-41ca-a141-b2575d6d1c5c"
+					(reference "#PWR01")
+					(unit 1)
+				)
+			)
+		)
+	)
+	(symbol
 		(lib_id "power:+3.3V")
 		(at 34.29 35.56 0)
@@
 	)
 	(symbol
-		(lib_id "171013801:VCC")
-		(at 208.28 22.86 0)
-		(unit 1)
-		(exclude_from_sim no)
-		(in_bom yes)
-		(on_board yes)
-		(dnp no)
-		(fields_autoplaced yes)
-		(property "Reference" "#PWR03"
-			(at 208.28 26.67 0)
-			(effects
-				(font
-					(size 1.27 1.27)
-				)
-				(hide yes)
-			)
-		)
-		(property "Value" "VCC"
-			(at 208.28 17.78 0)
-			(effects
-				(font
-					(size 1.27 1.27)
-				)
-			)
-		)
-		(property "Footprint" ""
-			(at 208.28 22.86 0)
-			(effects
-				(font
-					(size 1.27 1.27)
-				)
-				(hide yes)
-			)
-		)
-		(property "Datasheet" ""
-			(at 208.28 22.86 0)
-			(effects
-				(font
-					(size 1.27 1.27)
-				)
-				(hide yes)
-			)
-		)
-		(property "Description" "Power symbol creates a global label with name \"VCC\""
-			(at 208.28 22.86 0)
-			(effects
-				(font
-					(size 1.27 1.27)
-				)
-				(hide yes)
-			)
-		)
-		(pin "1"
-		)
-		(instances
-			(project ""
-				(path "/61133cf5-41c1-41ca-a141-b2575d6d1c5c"
-					(reference "#PWR03")
-					(unit 1)
-				)
-			)
-		)
-	)
-	(symbol
 		(lib_id "Device:R_Small")
 		(at 72.39 127 90)
@@
 					(unit 1)
 				)
-			)
-		)
-	)
-	(symbol
-		(lib_id "171013801:VCC")
-		(at 184.15 40.64 0)
-		(unit 1)
-		(exclude_from_sim no)
-		(in_bom yes)
-		(on_board yes)
-		(dnp no)
-		(fields_autoplaced yes)
-		(property "Reference" "#PWR01"
-			(at 184.15 44.45 0)
-			(effects
-				(font
-					(size 1.27 1.27)
-				)
-				(hide yes)
-			)
-		)
-		(property "Value" "VCC"
-			(at 184.15 35.56 0)
-			(effects
-				(font
-					(size 1.27 1.27)
-				)
-			)
-		)
-		(property "Footprint" ""
-			(at 184.15 40.64 0)
-			(effects
-				(font
-					(size 1.27 1.27)
-				)
-				(hide yes)
-			)
-		)
-		(property "Datasheet" ""
-			(at 184.15 40.64 0)
-			(effects
-				(font
-					(size 1.27 1.27)
-				)
-				(hide yes)
-			)
-		)
-		(property "Description" "Power symbol creates a global label with name \"VCC\""
-			(at 184.15 40.64 0)
-			(effects
-				(font
-					(size 1.27 1.27)
-				)
-				(hide yes)
-			)
-		)
-		(pin "1"
-		)
-		(instances
-			(project "PCB_Atlas_Gauntlet"
-				(path "/61133cf5-41c1-41ca-a141-b2575d6d1c5c"
-					(reference "#PWR01")
-					(unit 1)
-				)
