File: Hardware/PCB_Atlas_Gauntlet/PCB_Atlas_Gauntlet.kicad_pcb (KiCad board)
At the start: 2 copper layers, 40 parts, among them J1 Conn_01x02, J11 Conn_01x03, J13 Conn_01x03, J2 Conn_01x02, J3 Conn_01x03, J4 Conn_ST_STDC14, J5 Conn_01x03, J6 Conn_01x03, J7 Conn_01x03, J8 Conn_01x03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

Commit message: fix schematic
Parts:
- removed R22: 10k, Resistor_SMD:R_0402_1005Metric
- removed SW6: SW_Push, Connector_JST:JST_XH_B2B-XH-AM_1x02_P2.50mm_Vertical
- added C10: 10u, Capacitor_SMD:C_0603_1608Metric, F.Cu at (139.0, 91.3)
- added C11: 10u, Capacitor_SMD:C_0603_1608Metric, F.Cu at (139.0, 93.8)
- added C3: 47u, Capacitor_SMD:C_0805_2012Metric, F.Cu at (166.5, 69.2)
- added C4: 220u, Capacitor_SMD:CP_Elec_8x10.5, F.Cu at (151.6, 78.7)
- added C5: 10u, Capacitor_SMD:C_0603_1608Metric, F.Cu at (139.0, 78.8)
- added C6: 10u, Capacitor_SMD:C_0603_1608Metric, F.Cu at (139.0, 81.3)
- added C7: 10u, Capacitor_SMD:C_0603_1608Metric, F.Cu at (139.0, 83.8)
- added C8: 10u, Capacitor_SMD:C_0603_1608Metric, F.Cu at (139.0, 86.3)
- added C9: 10u, Capacitor_SMD:C_0603_1608Metric, F.Cu at (139.0, 88.8)
- C1: footprint Capacitor_SMD:C_0402_1005Metric -> Capacitor_SMD:C_0603_1608Metric
- J1: footprint Connector_AMASS:AMASS_XT30PW-M_1x02_P2.50mm_Horizontal -> Connector_AMASS:AMASS_XT30U-F_1x02_P5.0mm_Vertical
- SW1: footprint Connector_JST:JST_XH_B2B-XH-AM_1x02_P2.50mm_Vertical -> Button_Switch_SMD:SW_Push_1P1T_NO_CK_KSC7xxJ
- moved H4 111.8 mm to (50.0, 100.0)
- moved J5 63.6 mm to (128.5, 54.4)
- moved J6 63.6 mm to (128.5, 62.2)
- moved J7 63.6 mm to (128.5, 70.0)
- moved J8 63.6 mm to (128.5, 77.8)
- moved H2 61.5 mm to (100.0, 50.0)
- moved D10 54.2 mm to (162.3, 69.0)
- moved D11 54.2 mm to (162.3, 71.6)
- moved R18 48.2 mm to (146.4, 84.7)
- moved R19 48.2 mm to (146.4, 86.7)
- moved R20 48.2 mm to (146.4, 88.7)
- moved R21 48.2 mm to (146.4, 90.7)
- moved C12 47.5 mm to (165.2, 46.1)
- moved C14 47.5 mm to (165.2, 48.1)
- moved C15 47.5 mm to (165.2, 50.1)
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Connections:
- J11 pad 2: GPIO_LED_1 -> NEOPIXEL_PWM_1
- J13 pad 2: GPIO_LED_2 -> NEOPIXEL_PWM_2
- U3 pad 12: unconnected-(U3-PA6-Pad12) -> Servo_5
- U3 pad 14: /ADD_SEL_0 -> LED_0
- U3 pad 15: Servo_2 -> LED_1
- U3 pad 18: Servo_3 -> NEOPIXEL_PWM_1
- U3 pad 19: Servo_4 -> NEOPIXEL_PWM_2
- U3 pad 2: LED_0 -> Switch_On_Off
- U3 pad 21: Servo_5 -> unconnected-(U3-PA11-Pad21)
- U3 pad 25: /BTN_1 -> unconnected-(U3-PA15-Pad25)
- U3 pad 27: Switch_On_Off -> unconnected-(U3-PB4-Pad27)
- U3 pad 28: Button_Mode -> unconnected-(U3-PB5-Pad28)
- U3 pad 29: GPIO_LED_1 -> /VCP_TX
- U3 pad 3: LED_1 -> Button_Mode
- U3 pad 30: GPIO_LED_2 -> /VCP_RX
- U3 pad 31: /BOOT_0 -> GND
- U3 pad 6: /RCC_CLK_IN -> Servo_1
- U3 pad 7: Servo_1 -> Servo_2
- U3 pad 8: /VCP_TX -> Servo_3
- U3 pad 9: /VCP_RX -> Servo_4
Routing:
- net Servo_3: track 1.26 -> 0.00 mm
- net GND: track 0.99 -> 0.00 mm
- removed copper zone on F.Cu, net GND

Commit message: MAJ_PCB
Parts:
- moved C12 110.9 mm to (59.0, 77.8)
- moved C14 104.1 mm to (61.8, 59.4), turned to 90 degrees
- moved D10 101.7 mm to (62.4, 88.0), turned to 180 degrees
- moved U3 100.4 mm to (65.5, 78.0)
- moved J4 100.2 mm to (65.0, 67.0), turned to -90 degrees
- moved D11 98.2 mm to (65.5, 88.0), turned to 180 degrees
- moved C5 94.9 mm to (46.0, 59.7), turned to -90 degrees
- moved C19 94.1 mm to (75.0, 60.0), turned to 90 degrees
- moved C6 93.9 mm to (46.0, 68.2), turned to -90 degrees
- moved C7 93.3 mm to (46.0, 76.2), turned to -90 degrees
- moved R3 93.1 mm to (84.0, 92.0), turned to 180 degrees
- moved R1 93.1 mm to (84.0, 88.0), turned to 180 degrees
- moved C9 93.0 mm to (46.0, 92.0), turned to -90 degrees
- moved R2 93.0 mm to (84.0, 89.8)
- moved C8 93.0 mm to (46.0, 84.5), turned to -90 degrees
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Connections:
- C1 pad 1: VCC -> +5V
- C4 pad 1: VCC -> +5V
- J1 pad 1: VCC -> +5V
- U2 pad 4: VCC -> +5V
- U2 pad 5: VCC -> +5V
Routing:
- net +5V: track 0.00 -> 169.2 mm, vias 0 -> 2
- net +3.3V: track 0.00 -> 80.2 mm, vias 0 -> 2
- net /NRST: track 0.00 -> 45.4 mm, vias 0 -> 3
- net Switch_On_Off: track 0.00 -> 30.8 mm, vias 0 -> 2
- net NEOPIXEL_PWM_1: track 0.00 -> 28.9 mm
- net NEOPIXEL_PWM_2: track 0.00 -> 23.6 mm
- net Servo_1: track 0.00 -> 22.9 mm
- net Button_Mode: track 0.00 -> 20.7 mm
- net Servo_5: track 0.00 -> 16.7 mm
- net Servo_2: track 0.00 -> 16.2 mm
- net /VCP_RX: track 0.00 -> 11.6 mm
- net /SWDIO: track 0.00 -> 9.24 mm
- net Servo_4: track 0.00 -> 8.87 mm
- net Servo_3: track 0.00 -> 7.90 mm
- net Net-(R3-Pad2): track 0.00 -> 7.76 mm
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- added copper zone on B.Cu, net GND
- added copper zone on F.Cu, net GND
Other:
- board outline added: 45 x 60 mm

Commit message: MAJ PCB
Parts:
- moved C16 27.1 mm to (59.3, 78.4), turned to 180 degrees
- moved C17 26.7 mm to (60.7, 73.7), turned to 90 degrees
- moved C15 15.7 mm to (70.2, 82.4), turned to 90 degrees
- moved C18 15.4 mm to (71.5, 82.9), turned to -90 degrees
- moved R3 5.77 mm to (82.6, 86.4)
- moved R2 4.57 mm to (82.6, 85.4)
- moved R1 3.87 mm to (82.6, 84.4)
- moved C3 3.07 mm to (83.4, 76.7)
- moved C12 0.80 mm to (58.9, 77.0)
Routing:
- net Net-(R3-Pad2): track 7.76 -> 1.98 mm
- net Net-(R1-Pad2): track 6.85 -> 2.34 mm
- net Servo_5: track 16.7 -> 19.4 mm
- net Switch_On_Off: track 30.8 -> 33.1 mm
- net /SWCLK: track 7.61 -> 9.71 mm
- net +5V: track 169.2 -> 167.2 mm
- net NEOPIXEL_PWM_1: track 28.9 -> 30.7 mm
- net NEOPIXEL_PWM_2: track 23.6 -> 25.3 mm
- net Button_Mode: track 20.7 -> 21.6 mm
- net /SWDIO: track 9.24 -> 9.88 mm
- net /VCP_TX: track 6.84 -> 7.47 mm
- net Servo_4: track 8.87 -> 9.43 mm
- net GND: track 4.48 -> 3.94 mm, vias 6 -> 84
- net Servo_3: track 7.90 -> 8.43 mm
Other:
- board text added: "Maker 2425 Atlas Gauntlet Sédrenn"

Commit message: kjfv
Routing:
- net GND: vias 84 -> 88
